File: sch/counter/flip-flop.sch (KiCad schematic (older format))
At the start: 36 parts, among them Q1 Q_NMOS_GSD, Q2 Q_NMOS_GSD, Q3 Q_NMOS_GSD, Q4 Q_NMOS_GSD, Q5 Q_NMOS_GSD, Q6 Q_NMOS_GSD, Q7 Q_NMOS_GSD, Q8 Q_NMOS_GSD

Commit message: One flip-flop is placed on PCB
Parts:
- D10, D11, D12, D13, D14, D15, D16, D17, D18, D19, D20, D21, D22, D23, D24, D5, D6, D7, D8, D9: footprint (none) -> Diode_SMD:D_MiniMELF
- Q1, Q2, Q3, Q4, Q5, Q6, Q7, Q8: footprint (none) -> Package_TO_SOT_SMD:SOT-23
- R10, R11, R12, R5, R6, R7, R8, R9: footprint (none) -> Resistor_SMD:R_0805_2012Metric
