File: sch/decoder/decoder.kicad_pcb (KiCad board)
At the start: 2 copper layers, 53 x 91 mm, 166 parts, among them J1 In, J2 Out, J3 Power, Q1 2N7002, Q10 2N7002, Q11 2N7002, Q12 2N7002, Q2 2N7002, Q3 2N7002, Q4 2N7002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

Commit message: Decoder board finished
Other:
- board text added: "- +"
- board text added: "IN"
- board text added: "OUT"
