File: sch/decoder/decoder.sch (KiCad schematic (older format))
At the start: 142 parts, among them J1 In, J2 Out, J3 Power, Q1 2N7002, Q10 2N7002, Q11 2N7002, Q12 2N7002, Q2 2N7002, Q3 2N7002, Q4 2N7002, Q5 2N7002, Q6 2N7002, Q7 2N7002, Q8 2N7002, Q9 2N7002

Commit message: Decoder board added
Also schematics modified: added LEDs, configurable zero
Parts:
- removed D40, D41, D42, D43, D44, D45: D, symbol Device:D
- added D114, D115: D, Diode_SMD:D_MiniMELF, symbol Device:D
- added D116, D117, D118, D119, D120, D121, D40, D41, D42, D43, D44, D45: LED, LED_SMD:LED_0805_2012Metric, symbol Device:LED
- added H1, H2, H3, H4: MountingHole, MountingHole:MountingHole_3.2mm_M3_DIN965_Pad, symbol Mechanical:MountingHole
- added R13, R14, R15, R16, R17, R18, R19, R20, R21, R22, R23, R24: 50, Resistor_SMD:R_0805_2012Metric, symbol Device:R
- C1: footprint (none) -> Capacitor_SMD:C_0805_2012Metric
- C2: footprint (none) -> Capacitor_Tantalum_SMD:CP_EIA-3528-21_Kemet-B
- D1, D10, D100, D101, D102, D103, D104, D105, D106, D107, D108, D109, D11, D110, D111, D112, D113, D12, D13, D14, D15, D16, D17, D18, D19, D2, D20, D21, D22, D23, D24, D25, D26, D27, D28, D29, D3, D30, D31, D32, D33, D34, D35, D36, D37, D38, D39, D4, D46, D47, D48, D49, D5, D50, D51, D52, D53, D54, D55, D56, D57, D58, D59, D6, D60, D61, D62, D63, D64, D65, D66, D67, D68, D69, D7, D70, D71, D72, D73, D74, D75, D76, D77, D78, D79, D8, D80, D81, D82, D83, D84, D85, D86, D87, D88, D89, D9, D90, D91, D92, D93, D94, D95, D96, D97, D98, D99: footprint (none) -> Diode_SMD:D_MiniMELF
- J1, J2: footprint (none) -> Connector_IDC:IDC-Header_2x04_P2.54mm_Vertical
- J3: footprint (none) -> Connector_PinHeader_2.54mm:PinHeader_1x02_P2.54mm_Vertical
- Q1, Q10, Q11, Q12, Q2, Q3, Q4, Q5, Q6, Q7, Q8, Q9: footprint (none) -> Package_TO_SOT_SMD:SOT-23
- R1, R10, R11, R12, R2, R3, R4, R5, R6, R7, R8, R9: footprint (none) -> Resistor_SMD:R_0805_2012Metric
Connections:
- net VCC: now also D116.2 (A), D117.2 (A), D118.2 (A), D119.2 (A), D120.2 (A), D121.2 (A), D40.2 (A), D41.2 (A), D42.2 (A), D43.2 (A), D44.2 (A), D45.2 (A)
- net ~Sg: now also D114.2 (A)
- net ~Sten: now also D115.2 (A)
- net ~W0: now also D114.1 (K), D115.1 (K), R13.1
- net ~W1: now also R14.1
- net ~W10: now also R23.1
- net ~W11: now also R24.1
- net ~W2: now also R15.1
- net ~W3: now also R16.1
- net ~W4: now also R17.1
- net ~W5: now also R18.1
- net ~W6: now also R19.1
- net ~W7: now also R20.1
- net ~W8: now also R21.1
- net ~W9: now also R22.1
- new net: D44.1 (K), R17.2
- new net: D43.1 (K), R16.2
- new net: D45.1 (K), R18.2
- new net: D41.1 (K), R14.2
- new net: D40.1 (K), R13.2
- new net: D42.1 (K), R15.2
- new net: D120.1 (K), R23.2
- new net: D119.1 (K), R22.2
- new net: D121.1 (K), R24.2
- new net: D117.1 (K), R20.2
- new net: D116.1 (K), R19.2
- new net: D118.1 (K), R21.2
Other:
- note added: "Zero is configurable:\nonly necessary diodes should be installed"
- moved on the sheet: D106, D107, D108, D109, D110, D111, D112, D113, D26, D27, D28, D29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

Commit message: Added datasheets, set component values, calculated LED resistors
Parts:
- D1, D10, D100, D101, D102, D103, D104, D105, D106, D107, D108, D109, D11, D110, D111, D112, D113, D114, D115, D12, D13, D14, D15, D16, D17, D18, D19, D2, D20, D21, D22, D23, D24, D25, D26, D27, D28, D29, D3, D30, D31, D32, D33, D34, D35, D36, D37, D38, D39, D4, D46, D47, D48, D49, D5, D50, D51, D52, D53, D54, D55, D56, D57, D58, D59, D6, D60, D61, D62, D63, D64, D65, D66, D67, D68, D69, D7, D70, D71, D72, D73, D74, D75, D76, D77, D78, D79, D8, D80, D81, D82, D83, D84, D85, D86, D87, D88, D89, D9, D90, D91, D92, D93, D94, D95, D96, D97, D98, D99: value D -> LL103C
- R13, R14, R15, R16, R17, R18, R19, R20, R21, R22, R23, R24: value 50 -> 180
Other:
- note added: "The resistor values are specified for 1.8V 20mA LEDs"
