File: sch/display/display.sch (KiCad schematic (older format))
At the start: 49 parts, among them J1 S_Carry, J2 M_Carry, J3 Hour, J4 Second, J5 M_CLK, J6 H_CLK, J7 Minute10, J8 Minute1, J9 ~RST, SW1 M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

Commit message: 7-segment indicator footprint is added
Parts:
- C1: renamed from C?; footprint (none) -> Capacitor_SMD:C_0805_2012Metric
- C2: renamed from C1; footprint (none) -> Capacitor_SMD:CP_Elec_4x4.5
- C3: renamed from C2; footprint (none) -> Capacitor_SMD:C_0805_2012Metric
- J1, J2, J5, J6: footprint (none) -> Connector_PinHeader_2.54mm:PinHeader_1x02_P2.54mm_Vertical
- J10: renamed from J?; footprint (none) -> Connector_PinHeader_2.54mm:PinHeader_1x03_P2.54mm_Vertical
- J3, J7, J8: footprint (none) -> Connector_IDC:IDC-Header_2x04_P2.54mm_Vertical
- J4, J9: footprint (none) -> Connector_PinHeader_2.54mm:PinHeader_1x01_P2.54mm_Vertical
- Q1, Q2: renamed from Q?; footprint (none) -> Package_TO_SOT_SMD:SOT-23
- R1, R10, R11, R12, R13, R14, R15, R16, R17, R18, R19, R2, R20, R21, R22, R23, R24, R3, R4, R5, R6, R7, R8, R9: footprint (none) -> Resistor_SMD:R_0805_2012Metric
- R25, R26, R27: renamed from R?; footprint (none) -> Resistor_SMD:R_0805_2012Metric
- U1, U2, U3, U4: footprint Display_7Segment:KCSC02-105 -> lib:SA23-12EWA

Commit message: Button footprint added
Parts:
- SW1, SW2, SW3: footprint (none) -> lib:DTS-644
Changed lines of the file:
@@
 F 0 "SW3" H 7250 3185 50  0000 C CNN
 F 1 "Reset" H 7250 3094 50  0000 C CNN
-F 2 "" H 7250 3100 50  0001 C CNN
+F 2 "lib:DTS-644" H 7250 3100 50  0001 C CNN
 F 3 "" H 7250 3100 50  0001 C CNN
 	1    7250 2900
@@
 F 0 "SW1" H 1800 4835 50  0000 C CNN
 F 1 "M" H 1800 4744 50  0000 C CNN
-F 2 "" H 1800 4750 50  0001 C CNN
+F 2 "lib:DTS-644" H 1800 4750 50  0001 C CNN
 F 3 "" H 1800 4750 50  0001 C CNN
 	1    1800 4550
@@
 F 0 "SW2" H 1800 5785 50  0000 C CNN
 F 1 "H" H 1800 5694 50  0000 C CNN
-F 2 "" H 1800 5700 50  0001 C CNN
+F 2 "lib:DTS-644" H 1800 5700 50  0001 C CNN
 F 3 "" H 1800 5700 50  0001 C CNN
 	1    1800 5500

Commit message: Added datasheets, set component values, calculated LED resistors
Parts:
- J10: value Conn_01x03 -> Power
- R1, R11, R12, R13, R14, R15, R16, R17, R18, R19, R2, R20, R21, R22, R23, R24, R3, R4, R5, R6, R7, R8, R9: value 50 -> 15
- R10: value 50 -> 270
Connections:
- net +10V renamed VAA
Other:
- note added: "Resistor values are for VAA = 8.46 V (6 V AC transformer output)."
Changed lines of the file:
@@
 P 2750 2750
 F 0 "R1" V 2750 2200 50  0000 C CNN
-F 1 "50" V 2750 2350 50  0000 C CNN
+F 1 "15" V 2750 2350 50  0000 C CNN
 F 2 "Resistor_SMD:R_0805_2012Metric" V 2680 2750 50  0001 C CNN
 F 3 "~" H 2750 2750 50  0001 C CNN
@@
 P 2750 2850
 F 0 "R2" V 2750 2300 50  0000 C CNN
-F 1 "50" V 2750 2450 50  0000 C CNN
+F 1 "15" V 2750 2450 50  0000 C CNN
 F 2 "Resistor_SMD:R_0805_2012Metric" V 2680 2850 50  0001 C CNN
 F 3 "~" H 2750 2850 50  0001 C CNN
@@
 P 2750 2950
 F 0 "R3" V 2750 2400 50  0000 C CNN
-F 1 "50" V 2750 2550 50  0000 C CNN
+F 1 "15" V 2750 2550 50  0000 C CNN
 F 2 "Resistor_SMD:R_0805_2012Metric" V 2680 2950 50  0001 C CNN
 F 3 "~" H 2750 2950 50  0001 C CNN
@@
 P 2750 3050
 F 0 "R4" V 2750 2500 50  0000 C CNN
-F 1 "50" V 2750 2650 50  0000 C CNN
+F 1 "15" V 2750 2650 50  0000 C CNN
 F 2 "Resistor_SMD:R_0805_2012Metric" V 2680 3050 50  0001 C CNN
 F 3 "~" H 2750 3050 50  0001 C CNN
@@
 P 3550 2750
 F 0 "R5" V 3550 2200 50  0000 C CNN
-F 1 "50" V 3550 2350 50  0000 C CNN
+F 1 "15" V 3550 2350 50  0000 C CNN
 F 2 "Resistor_SMD:R_0805_2012Metric" V 3480 2750 50  0001 C CNN
 F 3 "~" H 3550 2750 50  0001 C CNN
@@
 P 3550 2850
 F 0 "R6" V 3550 2300 50  0000 C CNN
-F 1 "50" V 3550 2450 50  0000 C CNN
+F 1 "15" V 3550 2450 50  0000 C CNN
 F 2 "Resistor_SMD:R_0805_2012Metric" V 3480 2850 50  0001 C CNN
 F 3 "~" H 3550 2850 50  0001 C CNN
@@
 P 3550 2950
 F 0 "R7" V 3550 2400 50  0000 C CNN
-F 1 "50" V 3550 2550 50  0000 C CNN
+F 1 "15" V 3550 2550 50  0000 C CNN
 F 2 "Resistor_SMD:R_0805_2012Metric" V 3480 2950 50  0001 C CNN
 F 3 "~" H 3550 2950 50  0001 C CNN
@@
 P 3550 3050
 F 0 "R8" V 3550 2500 50  0000 C CNN
-F 1 "50" V 3550 2650 50  0000 C CNN
+F 1 "15" V 3550 2650 50  0000 C CNN
 F 2 "Resistor_SMD:R_0805_2012Metric" V 3480 3050 50  0001 C CNN
 F 3 "~" H 3550 3050 50  0001 C CNN
@@
 P 3550 3150
 F 0 "R9" V 3550 2600 50  0000 C CNN
-F 1 "50" V 3550 2750 50  0000 C CNN
+F 1 "15" V 3550 2750 50  0000 C CNN
 F 2 "Resistor_SMD:R_0805_2012Metric" V 3480 3150 50  0001 C CNN
 F 3 "~" H 3550 3150 50  0001 C CNN
@@
 P 5000 2750
 F 0 "R11" V 5000 2200 50  0000 C CNN
-F 1 "50" V 5000 2350 50  0000 C CNN
+F 1 "15" V 5000 2350 50  0000 C CNN
 F 2 "Resistor_SMD:R_0805_2012Metric" V 4930 2750 50  0001 C CNN
 F 3 "~" H 5000 2750 50  0001 C CNN
@@
 P 5000 2850
 F 0 "R12" V 5000 2300 50  0000 C CNN
-F 1 "50" V 5000 2450 50  0000 C CNN
+F 1 "15" V 5000 2450 50  0000 C CNN
 F 2 "Resistor_SMD:R_0805_2012Metric" V 4930 2850 50  0001 C CNN
 F 3 "~" H 5000 2850 50  0001 C CNN
@@
 P 5000 2950
 F 0 "R13" V 5000 2400 50  0000 C CNN
-F 1 "50" V 5000 2550 50  0000 C CNN
+F 1 "15" V 5000 2550 50  0000 C CNN
 F 2 "Resistor_SMD:R_0805_2012Metric" V 4930 2950 50  0001 C CNN
 F 3 "~" H 5000 2950 50  0001 C CNN
@@
 P 5000 3050
 F 0 "R14" V 5000 2500 50  0000 C CNN
-F 1 "50" V 5000 2650 50  0000 C CNN
+F 1 "15" V 5000 2650 50  0000 C CNN
 F 2 "Resistor_SMD:R_0805_2012Metric" V 4930 3050 50  0001 C CNN
 F 3 "~" H 5000 3050 50  0001 C CNN
@@
 P 5800 2750
 F 0 "R19" V 5800 2200 50  0000 C CNN
-F 1 "50" V 5800 2350 50  0000 C CNN
+F 1 "15" V 5800 2350 50  0000 C CNN
 F 2 "Resistor_SMD:R_0805_2012Metric" V 5730 2750 50  0001 C CNN
 F 3 "~" H 5800 2750 50  0001 C CNN
@@
 P 5800 2850
 F 0 "R20" V 5800 2300 50  0000 C CNN
-F 1 "50" V 5800 2450 50  0000 C CNN
+F 1 "15" V 5800 2450 50  0000 C CNN
 F 2 "Resistor_SMD:R_0805_2012Metric" V 5730 2850 50  0001 C CNN
 F 3 "~" H 5800 2850 50  0001 C CNN
@@
 P 5800 2950
 F 0 "R21" V 5800 2400 50  0000 C CNN
-F 1 "50" V 5800 2550 50  0000 C CNN
+F 1 "15" V 5800 2550 50  0000 C CNN
 F 2 "Resistor_SMD:R_0805_2012Metric" V 5730 2950 50  0001 C CNN
 F 3 "~" H 5800 2950 50  0001 C CNN
@@
 P 5000 3400
 F 0 "R15" V 5000 2850 50  0000 C CNN
-F 1 "50" V 5000 3000 50  0000 C CNN
+F 1 "15" V 5000 3000 50  0000 C CNN
 F 2 "Resistor_SMD:R_0805_2012Metric" V 4930 3400 50  0001 C CNN
 F 3 "~" H 5000 3400 50  0001 C CNN
@@
 P 5000 3500
 F 0 "R16" V 5000 2950 50  0000 C CNN
-F 1 "50" V 5000 3100 50  0000 C CNN
+F 1 "15" V 5000 3100 50  0000 C CNN
 F 2 "Resistor_SMD:R_0805_2012Metric" V 4930 3500 50  0001 C CNN
 F 3 "~" H 5000 3500 50  0001 C CNN
@@
 P 5000 3600
 F 0 "R17" V 5000 3050 50  0000 C CNN
-F 1 "50" V 5000 3200 50  0000 C CNN
+F 1 "15" V 5000 3200 50  0000 C CNN
 F 2 "Resistor_SMD:R_0805_2012Metric" V 4930 3600 50  0001 C CNN
 F 3 "~" H 5000 3600 50  0001 C CNN
@@
 P 5000 3700
 F 0 "R18" V 5000 3150 50  0000 C CNN
-F 1 "50" V 5000 3300 50  0000 C CNN
+F 1 "15" V 5000 3300 50  0000 C CNN
 F 2 "Resistor_SMD:R_0805_2012Metric" V 4930 3700 50  0001 C CNN
 F 3 "~" H 5000 3700 50  0001 C CNN
@@
 P 5800 3400
 F 0 "R22" V 5800 2850 50  0000 C CNN
-F 1 "50" V 5800 3000 50  0000 C CNN
+F 1 "15" V 5800 3000 50  0000 C CNN
 F 2 "Resistor_SMD:R_0805_2012Metric" V 5730 3400 50  0001 C CNN
 F 3 "~" H 5800 3400 50  0001 C CNN
@@
 P 5800 3500
 F 0 "R23" V 5800 2950 50  0000 C CNN
-F 1 "50" V 5800 3100 50  0000 C CNN
+F 1 "15" V 5800 3100 50  0000 C CNN
 F 2 "Resistor_SMD:R_0805_2012Metric" V 5730 3500 50  0001 C CNN
 F 3 "~" H 5800 3500 50  0001 C CNN
@@
 P 5800 3600
 F 0 "R24" V 5800 3050 50  0000 C CNN
-F 1 "50" V 5800 3200 50  0000 C CNN
+F 1 "15" V 5800 3200 50  0000 C CNN
 F 2 "Resistor_SMD:R_0805_2012Metric" V 5730 3600 50  0001 C CNN
 F 3 "~" H 5800 3600 50  0001 C CNN
@@
 Anode
 $Comp
-L power:+10V #PWR01
-U 1 1 5C131347
-P 1200 1200
-F 0 "#PWR01" H 1200 1050 50  0001 C CNN
-F 1 "+10V" V 1215 1328 50  0000 L CNN
-F 2 "" H 1200 1200 50  0001 C CNN
-F 3 "" H 1200 1200 50  0001 C CNN
-	1    1200 1200
-	0    -1   -1   0
-$EndComp
-$Comp
 L Switch:SW_Push_Dual SW3
 U 1 1 5C132B74
@@
 P 3550 3650
 F 0 "R10" V 3550 3050 50  0000 C CNN
-F 1 "50" V 3550 3200 50  0000 C CNN
+F 1 "270" V 3550 3200 50  0000 C CNN
 F 2 "Resistor_SMD:R_0805_2012Metric" V 3480 3650 50  0001 C CNN
 F 3 "~" H 3550 3650 50  0001 C CNN
@@
 	1    10050 5750
 	1    0    0    -1
-$EndComp
-$Comp
-L power:+10V #PWR018
-U 1 1 5C148274
-P 10050 5750
-F 0 "#PWR018" H 10050 5600 50  0001 C CNN
-F 1 "+10V" V 9950 5750 50  0000 L CNN
-F 2 "" H 10050 5750 50  0001 C CNN
-F 3 "" H 10050 5750 50  0001 C CNN
-	1    10050 5750
-	-1   0    0    1
 $EndComp
 $Comp
@@
 P 10000 950
 F 0 "J10" H 10080 992 50  0000 L CNN
-F 1 "Conn_01x03" H 10080 901 50  0000 L CNN
+F 1 "Power" H 10080 901 50  0000 L CNN
 F 2 "Connector_PinHeader_2.54mm:PinHeader_1x03_P2.54mm_Vertical" H 10000 950 50  0001 C CNN
 F 3 "~" H 10000 950 50  0001 C CNN
@@
 $EndComp
 $Comp
-L power:+10V #PWR016
-U 1 1 5C1625CC
+L power:VAA #PWR?
+U 1 1 5C32D65B
+P 1200 1200
+F 0 "#PWR?" H 1200 1050 50  0001 C CNN
+F 1 "VAA" V 1218 1327 50  0000 L CNN
+F 2 "" H 1200 1200 50  0001 C CNN
+F 3 "" H 1200 1200 50  0001 C CNN
+	1    1200 1200
+	0    -1   -1   0
+$EndComp
+$Comp
+L power:VAA #PWR?
+U 1 1 5C32D863
 P 9800 1050
-F 0 "#PWR016" H 9800 900 50  0001 C CNN
-F 1 "+10V" V 9815 1178 50  0000 L CNN
+F 0 "#PWR?" H 9800 900 50  0001 C CNN
+F 1 "VAA" V 9818 1177 50  0000 L CNN
 F 2 "" H 9800 1050 50  0001 C CNN
 F 3 "" H 9800 1050 50  0001 C CNN
@@
 	0    -1   -1   0
 $EndComp
+$Comp
+L power:VAA #PWR?
+U 1 1 5C32DB4E
+P 10050 5750
+F 0 "#PWR?" H 10050 5600 50  0001 C CNN
+F 1 "VAA" H 10050 5900 50  0000 C CNN
+F 2 "" H 10050 5750 50  0001 C CNN
+F 3 "" H 10050 5750 50  0001 C CNN
+	1    10050 5750
+	-1   0    0    1
+$EndComp
+Text Notes 5350 3850 2    50   ~ 0
+Resistor values are for VAA = 8.46 V (6 V AC transformer output).
 $EndSCHEMATC

Commit message: Display board, BOM updated
Parts:
- added H1, H2, H3, H4, H5, H6, H7, H8: MountingHole_Pad, MountingHole:MountingHole_3.2mm_M3_DIN965_Pad, symbol Mechanical:MountingHole_Pad
- C2: footprint Capacitor_SMD:CP_Elec_4x4.5 -> Capacitor_Tantalum_SMD:CP_EIA-3528-21_Kemet-B_Pad1.50x2.35mm_HandSolder
- U1, U2, U3, U4: footprint lib:SA23-12EWA -> lib:SA10-21HWA
Connections:
- net Anode is gone; now on net VAA: U1.3 (CA), U1.8 (CA), U2.3 (CA), U2.8 (CA), U3.3 (CA), U3.8 (CA), U4.3 (CA), U4.8 (CA)
- no-connect marks 10 -> 18
Changed lines of the file:
@@
 $Descr A4 11693 8268
 encoding utf-8
-Sheet 1 4
+Sheet 1 3
 Title ""
 Date ""
@@
 F 0 "U1" H 3550 2167 50  0000 C CNN
 F 1 "SA23-12EWA" H 3550 2076 50  0000 C CNN
-F 2 "lib:SA23-12EWA" H 3550 900 50  0001 C CNN
+F 2 "lib:SA10-21HWA" H 3550 900 50  0001 C CNN
 F 3 "http://www.kingbright.com/attachments/file/psearch/000/00/00/KCSA02-105(Ver.10A).pdf" H 3050 1975 50  0001 L CNN
 	1    3550 1500
@@
 F 0 "U2" H 4400 2167 50  0000 C CNN
 F 1 "SA23-12EWA" H 4400 2076 50  0000 C CNN
-F 2 "lib:SA23-12EWA" H 4400 900 50  0001 C CNN
+F 2 "lib:SA10-21HWA" H 4400 900 50  0001 C CNN
 F 3 "http://www.kingbright.com/attachments/file/psearch/000/00/00/KCSA02-105(Ver.10A).pdf" H 3900 1975 50  0001 L CNN
 	1    4400 1500
@@
 F 0 "U3" H 5250 2167 50  0000 C CNN
 F 1 "SA23-12EWA" H 5250 2076 50  0000 C CNN
-F 2 "lib:SA23-12EWA" H 5250 900 50  0001 C CNN
+F 2 "lib:SA10-21HWA" H 5250 900 50  0001 C CNN
 F 3 "http://www.kingbright.com/attachments/file/psearch/000/00/00/KCSA02-105(Ver.10A).pdf" H 4750 1975 50  0001 L CNN
 	1    5250 1500
@@
 F 0 "U4" H 6150 2167 50  0000 C CNN
 F 1 "SA23-12EWA" H 6150 2076 50  0000 C CNN
-F 2 "lib:SA23-12EWA" H 6150 900 50  0001 C CNN
+F 2 "lib:SA10-21HWA" H 6150 900 50  0001 C CNN
 F 3 "http://www.kingbright.com/attachments/file/psearch/000/00/00/KCSA02-105(Ver.10A).pdf" H 5650 1975 50  0001 L CNN
 	1    6150 1500
@@
 Text Label 4850 3700 2    50   ~ 0
 D4_g
-$Sheet
-S 1200 1050 750  650
-U 5C130866
-F0 "PWM" 50
-F1 "pwm.sch" 50
-F2 "Out" O R 1950 1200 50
-F3 "Vin" I L 1200 1200 50
-$EndSheet
 Wire Wire Line
 	1950 1200 2400 1200
@@
 F 0 "C2" H 8650 5600 50  0000 L CNN
 F 1 "10u x 16v" H 8400 5500 50  0000 L CNN
-F 2 "Capacitor_SMD:CP_Elec_4x4.5" H 8938 5450 50  0001 C CNN
+F 2 "Capacitor_Tantalum_SMD:CP_EIA-3528-21_Kemet-B_Pad1.50x2.35mm_HandSolder" H 8938 5450 50  0001 C CNN
 F 3 "~" H 8900 5600 50  0001 C CNN
 	1    8900 5600
@@
 $EndComp
 $Comp
-L power:VAA #PWR?
+L power:VAA #PWR01
 U 1 1 5C32D65B
-P 1200 1200
-F 0 "#PWR?" H 1200 1050 50  0001 C CNN
-F 1 "VAA" V 1218 1327 50  0000 L CNN
-F 2 "" H 1200 1200 50  0001 C CNN
-F 3 "" H 1200 1200 50  0001 C CNN
-	1    1200 1200
-	0    -1   -1   0
-$EndComp
-$Comp
-L power:VAA #PWR?
+P 1950 1200
+F 0 "#PWR01" H 1950 1050 50  0001 C CNN
+F 1 "VAA" V 1968 1327 50  0000 L CNN
+F 2 "" H 1950 1200 50  0001 C CNN
+F 3 "" H 1950 1200 50  0001 C CNN
+	1    1950 1200
+	0    -1   -1   0
+$EndComp
+$Comp
+L power:VAA #PWR016
 U 1 1 5C32D863
 P 9800 1050
-F 0 "#PWR?" H 9800 900 50  0001 C CNN
+F 0 "#PWR016" H 9800 900 50  0001 C CNN
 F 1 "VAA" V 9818 1177 50  0000 L CNN
 F 2 "" H 9800 1050 50  0001 C CNN
@@
 $EndComp
 $Comp
-L power:VAA #PWR?
+L power:VAA #PWR018
 U 1 1 5C32DB4E
 P 10050 5750
-F 0 "#PWR?" H 10050 5600 50  0001 C CNN
+F 0 "#PWR018" H 10050 5600 50  0001 C CNN
 F 1 "VAA" H 10050 5900 50  0000 C CNN
 F 2 "" H 10050 5750 50  0001 C CNN
@@
 Text Notes 5350 3850 2    50   ~ 0
 Resistor values are for VAA = 8.46 V (6 V AC transformer output).
+$Comp
+L Mechanical:MountingHole_Pad H2
+U 1 1 5C39FB43
+P 1500 7250
+F 0 "H2" H 1600 7255 50  0000 L CNN
+F 1 "MountingHole_Pad" H 1600 7210 50  0001 L CNN
+F 2 "MountingHole:MountingHole_3.2mm_M3_DIN965_Pad" H 1500 7250 50  0001 C CNN
+F 3 "~" H 1500 7250 50  0001 C CNN
+	1    1500 7250
+	1    0    0    -1
+$EndComp
+$Comp
+L Mechanical:MountingHole_Pad H5
+U 1 1 5C3A052D
+P 1850 7250
+F 0 "H5" H 1950 7255 50  0000 L CNN
+F 1 "MountingHole_Pad" H 1950 7210 50  0001 L CNN
+F 2 "MountingHole:MountingHole_3.2mm_M3_DIN965_Pad" H 1850 7250 50  0001 C CNN
+F 3 "~" H 1850 7250 50  0001 C CNN
+	1    1850 7250
+	1    0    0    -1
+$EndComp
+$Comp
+L Mechanical:MountingHole_Pad H8
+U 1 1 5C3A05AB
+P 2200 7250
+F 0 "H8" H 2300 7255 50  0000 L CNN
+F 1 "MountingHole_Pad" H 2300 7210 50  0001 L CNN
+F 2 "MountingHole:MountingHole_3.2mm_M3_DIN965_Pad" H 2200 7250 50  0001 C CNN
+F 3 "~" H 2200 7250 50  0001 C CNN
+	1    2200 7250
+	1    0    0    -1
+$EndComp
+$Comp
+L Mechanical:MountingHole_Pad H3
+U 1 1 5C3A0B33
+P 1500 7550
+F 0 "H3" H 1600 7555 50  0000 L CNN
+F 1 "MountingHole_Pad" H 1600 7510 50  0001 L CNN
+F 2 "MountingHole:MountingHole_3.2mm_M3_DIN965_Pad" H 1500 7550 50  0001 C CNN
+F 3 "~" H 1500 7550 50  0001 C CNN
+	1    1500 7550
+	1    0    0    -1
+$EndComp
+$Comp
+L Mechanical:MountingHole_Pad H6
+U 1 1 5C3A0BC8
+P 1850 7550
+F 0 "H6" H 1950 7555 50  0000 L CNN
+F 1 "MountingHole_Pad" H 1950 7510 50  0001 L CNN
+F 2 "MountingHole:MountingHole_3.2mm_M3_DIN965_Pad" H 1850 7550 50  0001 C CNN
+F 3 "~" H 1850 7550 50  0001 C CNN
+	1    1850 7550
+	1    0    0    -1
+$EndComp
+$Comp
+L Mechanical:MountingHole_Pad H7
+U 1 1 5C3A0DE0
+P 2200 6900
+F 0 "H7" H 2300 6905 50  0000 L CNN
+F 1 "MountingHole_Pad" H 2300 6860 50  0001 L CNN
+F 2 "MountingHole:MountingHole_3.2mm_M3_DIN965_Pad" H 2200 6900 50  0001 C CNN
+F 3 "~" H 2200 6900 50  0001 C CNN
+	1    2200 6900
+	1    0    0    -1
+$EndComp
+$Comp
+L Mechanical:MountingHole_Pad H4
+U 1 1 5C3A0E69
+P 1850 6900
+F 0 "H4" H 1950 6905 50  0000 L CNN
+F 1 "MountingHole_Pad" H 1950 6860 50  0001 L CNN
+F 2 "MountingHole:MountingHole_3.2mm_M3_DIN965_Pad" H 1850 6900 50  0001 C CNN
+F 3 "~" H 1850 6900 50  0001 C CNN
+	1    1850 6900
+	1    0    0    -1
+$EndComp
+$Comp
+L Mechanical:MountingHole_Pad H1
+U 1 1 5C3A0EF4
+P 1500 6900
+F 0 "H1" H 1600 6905 50  0000 L CNN
+F 1 "MountingHole_Pad" H 1600 6860 50  0001 L CNN
+F 2 "MountingHole:MountingHole_3.2mm_M3_DIN965_Pad" H 1500 6900 50  0001 C CNN
+F 3 "~" H 1500 6900 50  0001 C CNN
+	1    1500 6900
+	1    0    0    -1
+$EndComp
+NoConn ~ 1500 7000
+NoConn ~ 1850 7000
+NoConn ~ 2200 7000
+NoConn ~ 1850 7650
+NoConn ~ 1500 7650
+NoConn ~ 1500 7350
+NoConn ~ 1850 7350
+NoConn ~ 2200 7350
 $EndSCHEMATC
