File: sch/power/power.sch (KiCad schematic (older format))
At the start: 31 parts, among them J1 Sec_1A, J10 5V, J11 5V, J12 5V, J13 5V, J14 5V, J15 5V, J16 5V, J17 5V, J18 5V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

Commit message: Power supply board
Parts:
- added C4, C5: 0.1u, Capacitor_SMD:C_0805_2012Metric, symbol Device:C
- added H1, H2, H3, H4: MountingHole_Pad, MountingHole:MountingHole_3.2mm_M3_DIN965_Pad, symbol Mechanical:MountingHole_Pad
- added J19: Conn_01x03, Connector_PinHeader_2.54mm:PinHeader_1x03_P2.54mm_Vertical, symbol Connector_Generic:Conn_01x03
- added Q3: Q_NMOS_GSD, Package_TO_SOT_SMD:SOT-23, symbol Device:Q_NMOS_GSD
- added R2: 20k, Resistor_SMD:R_0805_2012Metric, symbol Device:R
- C1: value CP -> 1000u 10v; footprint (none) -> Capacitor_SMD:CP_Elec_10x10
- C2: footprint (none) -> Capacitor_SMD:CP_Elec_6.3x5.4
- C3: footprint (none) -> Capacitor_SMD:CP_Elec_8x10.5
- D1, D2, D3, D4: value D -> 1N5822; footprint (none) -> Diode_THT:D_DO-201AD_P12.70mm_Horizontal
- D5: footprint (none) -> Diode_THT:D_DO-201AD_P12.70mm_Horizontal
- J1, J2, J3, J4: footprint (none) -> Connector_Wire:SolderWirePad_1x01_Drill1.5mm
- J10, J11, J12, J13, J14, J15, J16, J17, J18, J5, J6, J7, J9: footprint (none) -> Connector_PinHeader_2.54mm:PinHeader_1x02_P2.54mm_Vertical
- J8: footprint (none) -> Connector_PinHeader_2.54mm:PinHeader_1x03_P2.54mm_Vertical
- L1: footprint (none) -> Inductor_SMD:L_Wuerth_WE-PD-Typ-LS_Handsoldering
- Q1, Q2: footprint (none) -> Package_TO_SOT_SMD:SOT-23
- R1: footprint (none) -> Resistor_SMD:R_0805_2012Metric
Connections:
- net +10V: now also J19.3 (Pin_3)
- net CLK: now also Q2.3 (D), Q3.1 (G), R2.2; no longer Q1.3 (D), Q2.1 (G), R1.2
- net GND: now also C4.2, C5.2, J19.2 (Pin_2), Q3.2 (S)
- net VCC: now also C4.1, C5.1, J19.1 (Pin_1), R2.1
- net ~CLK: now also Q3.3 (D); no longer Q2.3 (D)
- net Sec_A: now reaches D2.2 (A), D4.1 (K), J1.1 (Pin_1), J2.1 (Pin_1)
- net Sec_A: now also Q1.1 (G)
- net Sec_B: now reaches D1.2 (A), D3.1 (K), J3.1 (Pin_1), J4.1 (Pin_1)
- net Sec_B: no longer Q1.1 (G)
- net LM_out: now reaches D5.1 (K), L1.1, U1.2 (OUT)
- new net: Q1.3 (D), Q2.1 (G), R1.2
- no-connect marks 0 -> 4
